Commit message: added sim stuff. movement transferring properly to rviz

File: src/plum/description/robot_core.xacro (robot description, xacro)
@@ -45,5 +45,5 @@
     </link>
     <gazebo reference="chassis">
-        <material>Gazebo/Black</material>
+        <material>Gazebo/White</material>
     </gazebo>
     <!-- LEFT WHEEL LINK -->
@@ -71,5 +71,5 @@
     </link>
     <gazebo reference="left_wheel">
-        <material>Gazebo/Blue</material>
+        <material>Gazebo/Black</material>
     </gazebo>
     <!-- RIGHT WHEEL LINK -->
@@ -78,5 +78,5 @@
         <child link="right_wheel"/>
         <origin xyz="0 -0.15 0" rpy="${pi/2} 0 0" />
-        <axis xyz="0 0 1"/>
+        <axis xyz="0 0 -1"/>
     </joint>
     <link name="right_wheel">
