Commit message: slam toolbox mapping is working and publishing to rviz in SIM. map only smears when moving quickly. slam tb is launched via online_async.launch

File: src/plum/description/lidar.xacro (robot description, xacro)
@@ -27,5 +27,5 @@
             <pose> 0 0 0 0 0 0 </pose>
             <visualize>true</visualize>
-            <update_rate>10</update_rate>
+            <update_rate>30</update_rate>
             <ray>
                 <scan>
@@ -37,6 +37,6 @@
                 </scan>
                 <range>
-                    <min>0.3</min>
-                    <max>12</max>
+                    <min>0.1</min>
+                    <max>6</max>
                 </range>
             </ray>

File: src/plum/description/robot_core.xacro (robot description, xacro)
@@ -19,4 +19,12 @@
     <!-- BASE LINK -->
     <link name="base_link">
+    </link>
+    <!-- BASE_FOOTPRINT LINK -->
+    <joint name="base_footprint_joint" type="fixed">
+        <parent link="base_link"/>
+        <child link="base_footprint"/>
+        <origin xyz="0 0 0" rpy="0 0 0"/>
+    </joint>
+    <link name="base_footprint">
     </link>
     <!-- CHASSIS LINK -->
